File: latch.kicad_sch (KiCad schematic)
At the start: 16 parts, among them U1 74LS273, U2 74LS273, U3 74LS273, U4 74LS273, U5 74LS273, U6 74LS273, U7 74LS273, U8 74LS273

Commit message: Current progress.  Working on laying out the latched bus.
Parts:
- C10: renamed from C7; footprint (none) -> Capacitor_SMD:C_0805_2012Metric_Pad1.18x1.45mm_HandSolder
- C11: renamed from C8; footprint (none) -> Capacitor_SMD:C_0805_2012Metric_Pad1.18x1.45mm_HandSolder
- C4: renamed from C1; footprint (none) -> Capacitor_SMD:C_0805_2012Metric_Pad1.18x1.45mm_HandSolder
- C5: renamed from C2; footprint (none) -> Capacitor_SMD:C_0805_2012Metric_Pad1.18x1.45mm_HandSolder
- C6: renamed from C3; footprint (none) -> Capacitor_SMD:C_0805_2012Metric_Pad1.18x1.45mm_HandSolder
- C7: renamed from C4; footprint (none) -> Capacitor_SMD:C_0805_2012Metric_Pad1.18x1.45mm_HandSolder
- C8: renamed from C5; footprint (none) -> Capacitor_SMD:C_0805_2012Metric_Pad1.18x1.45mm_HandSolder
- C9: renamed from C6; footprint (none) -> Capacitor_SMD:C_0805_2012Metric_Pad1.18x1.45mm_HandSolder
- U10: renamed from U7; footprint (none) -> Package_SO:SOIC-20W_7.5x12.8mm_P1.27mm
- U11: renamed from U8; footprint (none) -> Package_SO:SOIC-20W_7.5x12.8mm_P1.27mm
- U4: renamed from U1; footprint (none) -> Package_SO:SOIC-20W_7.5x12.8mm_P1.27mm
- U5: renamed from U2; footprint (none) -> Package_SO:SOIC-20W_7.5x12.8mm_P1.27mm
- U6: renamed from U3; footprint (none) -> Package_SO:SOIC-20W_7.5x12.8mm_P1.27mm
- U7: renamed from U4; footprint (none) -> Package_SO:SOIC-20W_7.5x12.8mm_P1.27mm
- U8: renamed from U5; footprint (none) -> Package_SO:SOIC-20W_7.5x12.8mm_P1.27mm
- U9: renamed from U6; footprint (none) -> Package_SO:SOIC-20W_7.5x12.8mm_P1.27mm
Connections:
- net latched00 renamed latched0
- net latched01 renamed latched1
- net latched02 renamed latched2
- net latched03 renamed latched3
- net latched04 renamed latched4
- net latched05 renamed latched5
- net latched06 renamed latched6
- net latched07 renamed latched7
- net latched08 renamed latched8
- net latched09 renamed latched9
- net write00 renamed write0
- net write01 renamed write1
- net write02 renamed write2
- net write03 renamed write3
- net write04 renamed write4
- net write05 renamed write5
- net write06 renamed write6
- net write07 renamed write7
- net write08 renamed write8
- net write09 renamed write9
- net ~{RST} renamed ~{ZRST}

Commit message: Moar progress.  Working on the write in latch.
Connections:
- net latched0: now also U4.9 (Q3); no longer U4.2 (Q0)
- net latched1: now also U4.6 (Q2); no longer U4.5 (Q1)
- net latched10: now also U5.5 (Q1); no longer U5.6 (Q2)
- net latched11: now also U5.2 (Q0); no longer U5.9 (Q3)
- net latched12: now also U5.19 (Q7); no longer U5.12 (Q4)
- net latched13: now also U5.16 (Q6); no longer U5.15 (Q5)
- net latched14: now also U5.15 (Q5); no longer U5.16 (Q6)
- net latched15: now also U5.12 (Q4); no longer U5.19 (Q7)
- net latched16: now also U6.9 (Q3); no longer U6.2 (Q0)
- net latched17: now also U6.6 (Q2); no longer U6.5 (Q1)
- net latched18: now also U6.5 (Q1); no longer U6.6 (Q2)
- net latched19: now also U6.2 (Q0); no longer U6.9 (Q3)
- net latched2: now also U4.5 (Q1); no longer U4.6 (Q2)
- net latched20: now also U6.19 (Q7); no longer U6.12 (Q4)
- net latched21: now also U6.16 (Q6); no longer U6.15 (Q5)
- net latched22: now also U6.15 (Q5); no longer U6.16 (Q6)
- net latched23: now also U6.12 (Q4); no longer U6.19 (Q7)
- net latched24: now also U7.9 (Q3); no longer U7.2 (Q0)
- net latched25: now also U7.6 (Q2); no longer U7.5 (Q1)
- net latched26: now also U7.5 (Q1); no longer U7.6 (Q2)
- net latched27: now also U7.2 (Q0); no longer U7.9 (Q3)
- net latched28: now also U7.19 (Q7); no longer U7.12 (Q4)
- net latched29: now also U7.16 (Q6); no longer U7.15 (Q5)
- net latched3: now also U4.2 (Q0); no longer U4.9 (Q3)
- net latched30: now also U7.15 (Q5); no longer U7.16 (Q6)
- net latched31: now also U7.12 (Q4); no longer U7.19 (Q7)
- net latched32: now also U8.12 (Q4); no longer U8.2 (Q0)
- net latched33: now also U8.15 (Q5); no longer U8.5 (Q1)
- net latched34: now also U8.16 (Q6); no longer U8.6 (Q2)
- net latched35: now also U8.19 (Q7); no longer U8.9 (Q3)
- net latched36: now also U8.2 (Q0); no longer U8.12 (Q4)
- net latched37: now also U8.5 (Q1); no longer U8.15 (Q5)
- net latched38: now also U8.6 (Q2); no longer U8.16 (Q6)
- net latched39: now also U8.9 (Q3); no longer U8.19 (Q7)
- net latched4: now also U4.19 (Q7); no longer U4.12 (Q4)
- net latched40: now also U9.12 (Q4); no longer U9.2 (Q0)
- net latched41: now also U9.15 (Q5); no longer U9.5 (Q1)
- net latched42: now also U9.16 (Q6); no longer U9.6 (Q2)
- net latched43: now also U9.19 (Q7); no longer U9.9 (Q3)
- net latched44: now also U9.2 (Q0); no longer U9.12 (Q4)
- net latched45: now also U9.5 (Q1); no longer U9.15 (Q5)
- net latched46: now also U9.6 (Q2); no longer U9.16 (Q6)
- net latched47: now also U9.9 (Q3); no longer U9.19 (Q7)
- net latched48: now also U10.12 (Q4); no longer U10.2 (Q0)
- net latched49: now also U10.15 (Q5); no longer U10.5 (Q1)
- net latched5: now also U4.16 (Q6); no longer U4.15 (Q5)
- net latched50: now also U10.16 (Q6); no longer U10.6 (Q2)
- net latched51: now also U10.19 (Q7); no longer U10.9 (Q3)
- net latched52: now also U10.2 (Q0); no longer U10.12 (Q4)
- net latched53: now also U10.5 (Q1); no longer U10.15 (Q5)
- net latched54: now also U10.6 (Q2); no longer U10.16 (Q6)
- net latched55: now also U10.9 (Q3); no longer U10.19 (Q7)
- net latched56: now also U11.12 (Q4); no longer U11.2 (Q0)
- net latched57: now also U11.15 (Q5); no longer U11.5 (Q1)
- net latched58: now also U11.16 (Q6); no longer U11.6 (Q2)
- net latched59: now also U11.19 (Q7); no longer U11.9 (Q3)
- net latched6: now also U4.15 (Q5); no longer U4.16 (Q6)
- net latched60: now also U11.2 (Q0); no longer U11.12 (Q4)
- net latched61: now also U11.5 (Q1); no longer U11.15 (Q5)
- net latched62: now also U11.6 (Q2); no longer U11.16 (Q6)
- net latched63: now also U11.9 (Q3); no longer U11.19 (Q7)
- net latched7: now also U4.12 (Q4); no longer U4.19 (Q7)
- net latched8: now also U5.9 (Q3); no longer U5.2 (Q0)
- net latched9: now also U5.6 (Q2); no longer U5.5 (Q1)
- net write0: now also U4.8 (D3); no longer U4.3 (D0)
- net write1: now also U4.7 (D2); no longer U4.4 (D1)
- net write10: now also U5.4 (D1); no longer U5.7 (D2)
- net write11: now also U5.3 (D0); no longer U5.8 (D3)
- net write12: now also U5.18 (D7); no longer U5.13 (D4)
- net write13: now also U5.17 (D6); no longer U5.14 (D5)
- net write14: now also U5.14 (D5); no longer U5.17 (D6)
- net write15: now also U5.13 (D4); no longer U5.18 (D7)
- net write16: now also U6.8 (D3); no longer U6.3 (D0)
- net write17: now also U6.7 (D2); no longer U6.4 (D1)
- net write18: now also U6.4 (D1); no longer U6.7 (D2)
- net write19: now also U6.3 (D0); no longer U6.8 (D3)
- net write2: now also U4.4 (D1); no longer U4.7 (D2)
- net write20: now also U6.18 (D7); no longer U6.13 (D4)
- net write21: now also U6.17 (D6); no longer U6.14 (D5)
- net write22: now also U6.14 (D5); no longer U6.17 (D6)
- net write23: now also U6.13 (D4); no longer U6.18 (D7)
- net write24: now also U7.8 (D3); no longer U7.3 (D0)
- net write25: now also U7.7 (D2); no longer U7.4 (D1)
- net write26: now also U7.4 (D1); no longer U7.7 (D2)
- net write27: now also U7.3 (D0); no longer U7.8 (D3)
- net write28: now also U7.18 (D7); no longer U7.13 (D4)
- net write29: now also U7.17 (D6); no longer U7.14 (D5)
- net write3: now also U4.3 (D0); no longer U4.8 (D3)
- net write30: now also U7.14 (D5); no longer U7.17 (D6)
- net write31: now also U7.13 (D4); no longer U7.18 (D7)
- net write32: now also U8.13 (D4); no longer U8.3 (D0)
- net write33: now also U8.14 (D5); no longer U8.4 (D1)
- net write34: now also U8.17 (D6); no longer U8.7 (D2)
- net write35: now also U8.18 (D7); no longer U8.8 (D3)
- net write36: now also U8.3 (D0); no longer U8.13 (D4)
- net write37: now also U8.4 (D1); no longer U8.14 (D5)
- net write38: now also U8.7 (D2); no longer U8.17 (D6)
- net write39: now also U8.8 (D3); no longer U8.18 (D7)
- net write4: now also U4.18 (D7); no longer U4.13 (D4)
- net write40: now also U9.13 (D4); no longer U9.3 (D0)
- net write41: now also U9.14 (D5); no longer U9.4 (D1)
- net write42: now also U9.17 (D6); no longer U9.7 (D2)
- net write43: now also U9.18 (D7); no longer U9.8 (D3)
- net write44: now also U9.3 (D0); no longer U9.13 (D4)
- net write45: now also U9.4 (D1); no longer U9.14 (D5)
- net write46: now also U9.7 (D2); no longer U9.17 (D6)
- net write47: now also U9.8 (D3); no longer U9.18 (D7)
- net write48: now also U10.13 (D4); no longer U10.3 (D0)
- net write49: now also U10.14 (D5); no longer U10.4 (D1)
- net write5: now also U4.17 (D6); no longer U4.14 (D5)
- net write50: now also U10.17 (D6); no longer U10.7 (D2)
- net write51: now also U10.18 (D7); no longer U10.8 (D3)
- net write52: now also U10.3 (D0); no longer U10.13 (D4)
- net write53: now also U10.4 (D1); no longer U10.14 (D5)
- net write54: now also U10.7 (D2); no longer U10.17 (D6)
- net write55: now also U10.8 (D3); no longer U10.18 (D7)
- net write56: now also U11.13 (D4); no longer U11.3 (D0)
- net write57: now also U11.14 (D5); no longer U11.4 (D1)
- net write58: now also U11.17 (D6); no longer U11.7 (D2)
- net write59: now also U11.18 (D7); no longer U11.8 (D3)
- net write6: now also U4.14 (D5); no longer U4.17 (D6)
- net write60: now also U11.3 (D0); no longer U11.13 (D4)
- net write61: now also U11.4 (D1); no longer U11.14 (D5)
- net write62: now also U11.7 (D2); no longer U11.17 (D6)
- net write63: now also U11.8 (D3); no longer U11.18 (D7)
- net write7: now also U4.13 (D4); no longer U4.18 (D7)
- net write8: now also U5.8 (D3); no longer U5.3 (D0)
- net write9: now also U5.7 (D2); no longer U5.4 (D1)
