File: kdrv-discrete-pcb-register.kicad_pcb (KiCad board)
At the start: 2 copper layers, 284.3 x 41.5 mm, 3 parts, among them J1 Bus_PCI_Express_x16, J2 Bus_PCI_Express_x16, J3 Bus_PCI_Express_x16

Commit message: Current progress.  Working on laying out the latched bus.
Parts:
- added C1: 100 nF, Capacitor_SMD:C_0805_2012Metric_Pad1.18x1.45mm_HandSolder, B.Cu at (253.0, 155.0)
- added C10: 100 nF, Capacitor_SMD:C_0805_2012Metric_Pad1.18x1.45mm_HandSolder, B.Cu at (343.0, 127.1)
- added C11: 100 nF, Capacitor_SMD:C_0805_2012Metric_Pad1.18x1.45mm_HandSolder, B.Cu at (343.0, 130.1)
- added C12: 100 nF, Capacitor_SMD:C_0805_2012Metric_Pad1.18x1.45mm_HandSolder, B.Cu at (-3.54, 80.0)
- added C13: 100 nF, Capacitor_SMD:C_0805_2012Metric_Pad1.18x1.45mm_HandSolder, B.Cu at (-3.54, 83.0)
- added C14: 100 nF, Capacitor_SMD:C_0805_2012Metric_Pad1.18x1.45mm_HandSolder, B.Cu at (-3.54, 86.0)
- added C15: 100 nF, Capacitor_SMD:C_0805_2012Metric_Pad1.18x1.45mm_HandSolder, B.Cu at (-3.54, 89.0)
- added C16: 100 nF, Capacitor_SMD:C_0805_2012Metric_Pad1.18x1.45mm_HandSolder, B.Cu at (-3.54, 92.0)
- added C17: 100 nF, Capacitor_SMD:C_0805_2012Metric_Pad1.18x1.45mm_HandSolder, B.Cu at (-8.35, 80.0)
- added C18: 100 nF, Capacitor_SMD:C_0805_2012Metric_Pad1.18x1.45mm_HandSolder, B.Cu at (-8.35, 83.0)
- added C19: 100 nF, Capacitor_SMD:C_0805_2012Metric_Pad1.18x1.45mm_HandSolder, B.Cu at (-8.35, 86.0)
- added C2: 100 nF, Capacitor_SMD:C_0805_2012Metric_Pad1.18x1.45mm_HandSolder, B.Cu at (253.0, 158.0)
- added C20: 100 nF, Capacitor_SMD:C_0805_2012Metric_Pad1.18x1.45mm_HandSolder, B.Cu at (-8.35, 89.0)
- added C21: 100 nF, Capacitor_SMD:C_0805_2012Metric_Pad1.18x1.45mm_HandSolder, B.Cu at (-8.35, 92.0)
- added C22: 100 nF, Capacitor_SMD:C_0805_2012Metric_Pad1.18x1.45mm_HandSolder, B.Cu at (157.0, 151.5)
- added C23: 100 nF, Capacitor_SMD:C_0805_2012Metric_Pad1.18x1.45mm_HandSolder, B.Cu at (157.0, 154.5)
- added C24: 100 nF, Capacitor_SMD:C_0805_2012Metric_Pad1.18x1.45mm_HandSolder, B.Cu at (157.0, 157.5)
- added C25: 100 nF, Capacitor_SMD:C_0805_2012Metric_Pad1.18x1.45mm_HandSolder, B.Cu at (157.0, 160.5)
- added C26: 100 nF, Capacitor_SMD:C_0805_2012Metric_Pad1.18x1.45mm_HandSolder, B.Cu at (157.0, 163.5)
- added C27: 100 nF, Capacitor_SMD:C_0805_2012Metric_Pad1.18x1.45mm_HandSolder, B.Cu at (152.2, 151.5)
- added C28: 100 nF, Capacitor_SMD:C_0805_2012Metric_Pad1.18x1.45mm_HandSolder, B.Cu at (152.2, 154.5)
- added C29: 100 nF, Capacitor_SMD:C_0805_2012Metric_Pad1.18x1.45mm_HandSolder, B.Cu at (152.2, 157.5)
- added C3: 100 nF, Capacitor_SMD:C_0805_2012Metric_Pad1.18x1.45mm_HandSolder, B.Cu at (253.0, 161.0)
- added C30: 100 nF, Capacitor_SMD:C_0805_2012Metric_Pad1.18x1.45mm_HandSolder, B.Cu at (152.2, 160.5)
- added C31: 100 nF, Capacitor_SMD:C_0805_2012Metric_Pad1.18x1.45mm_HandSolder, B.Cu at (152.2, 163.5)
- added C4: 100 nF, Capacitor_SMD:C_0805_2012Metric_Pad1.18x1.45mm_HandSolder, B.Cu at (343.0, 109.0)
- added C5: 100 nF, Capacitor_SMD:C_0805_2012Metric_Pad1.18x1.45mm_HandSolder, B.Cu at (343.0, 112.0)
- added C6: 100 nF, Capacitor_SMD:C_0805_2012Metric_Pad1.18x1.45mm_HandSolder, B.Cu at (343.0, 115.0)
- added C7: 100 nF, Capacitor_SMD:C_0805_2012Metric_Pad1.18x1.45mm_HandSolder, B.Cu at (343.0, 118.0)
- added C8: 100 nF, Capacitor_SMD:C_0805_2012Metric_Pad1.18x1.45mm_HandSolder, B.Cu at (343.0, 121.0)
- added C9: 100 nF, Capacitor_SMD:C_0805_2012Metric_Pad1.18x1.45mm_HandSolder, B.Cu at (343.0, 124.0)
- added D1: LED 0603 0605 0805 Right Angle Yellow Amber Green, LED_SMD:LED_0805_2012Metric_Pad1.15x1.40mm_HandSolder, F.Cu at (72.0, -140.2)
- added D10: LED, LED_SMD:LED_0805_2012Metric_Pad1.15x1.40mm_HandSolder, F.Cu at (108.0, -140.2)
- added D11: LED, LED_SMD:LED_0805_2012Metric_Pad1.15x1.40mm_HandSolder, F.Cu at (112.0, -140.2)
- added D12: LED, LED_SMD:LED_0805_2012Metric_Pad1.15x1.40mm_HandSolder, F.Cu at (116.0, -140.2)
- added D13: LED, LED_SMD:LED_0805_2012Metric_Pad1.15x1.40mm_HandSolder, F.Cu at (120.0, -140.2)
- added D14: LED, LED_SMD:LED_0805_2012Metric_Pad1.15x1.40mm_HandSolder, F.Cu at (124.0, -140.2)
- added D15: LED, LED_SMD:LED_0805_2012Metric_Pad1.15x1.40mm_HandSolder, F.Cu at (128.0, -140.2)
- added D16: LED, LED_SMD:LED_0805_2012Metric_Pad1.15x1.40mm_HandSolder, F.Cu at (132.0, -140.2)
- added D17: LED, LED_SMD:LED_0805_2012Metric_Pad1.15x1.40mm_HandSolder, F.Cu at (136.0, -140.2)
- added D18: LED, LED_SMD:LED_0805_2012Metric_Pad1.15x1.40mm_HandSolder, F.Cu at (140.0, -140.2)
- added D19: LED, LED_SMD:LED_0805_2012Metric_Pad1.15x1.40mm_HandSolder, F.Cu at (144.0, -140.2)
- added D2: LED, LED_SMD:LED_0805_2012Metric_Pad1.15x1.40mm_HandSolder, F.Cu at (76.0, -140.2)
- added D20: LED, LED_SMD:LED_0805_2012Metric_Pad1.15x1.40mm_HandSolder, F.Cu at (148.0, -140.2)
- added D21: LED, LED_SMD:LED_0805_2012Metric_Pad1.15x1.40mm_HandSolder, F.Cu at (152.0, -140.2)
- added D22: LED, LED_SMD:LED_0805_2012Metric_Pad1.15x1.40mm_HandSolder, F.Cu at (156.0, -140.2)
- added D23: LED, LED_SMD:LED_0805_2012Metric_Pad1.15x1.40mm_HandSolder, F.Cu at (160.0, -140.2)
- added D24: LED, LED_SMD:LED_0805_2012Metric_Pad1.15x1.40mm_HandSolder, F.Cu at (163.9, -140.2)
- added D25: LED, LED_SMD:LED_0805_2012Metric_Pad1.15x1.40mm_HandSolder, F.Cu at (167.9, -140.2)
- added D26: LED, LED_SMD:LED_0805_2012Metric_Pad1.15x1.40mm_HandSolder, F.Cu at (171.9, -140.2)
- added D27: LED, LED_SMD:LED_0805_2012Metric_Pad1.15x1.40mm_HandSolder, F.Cu at (175.9, -140.2)
- added D28: LED, LED_SMD:LED_0805_2012Metric_Pad1.15x1.40mm_HandSolder, F.Cu at (179.9, -140.2)
- added D29: LED, LED_SMD:LED_0805_2012Metric_Pad1.15x1.40mm_HandSolder, F.Cu at (183.9, -140.2)
- added D3: LED, LED_SMD:LED_0805_2012Metric_Pad1.15x1.40mm_HandSolder, F.Cu at (80.0, -140.2)
- added D30: LED, LED_SMD:LED_0805_2012Metric_Pad1.15x1.40mm_HandSolder, F.Cu at (187.9, -140.2)
- added D31: LED, LED_SMD:LED_0805_2012Metric_Pad1.15x1.40mm_HandSolder, F.Cu at (191.8, -140.2)
- added D32: LED, LED_SMD:LED_0805_2012Metric_Pad1.15x1.40mm_HandSolder, F.Cu at (195.8, -140.2)
- added D33: LED, LED_SMD:LED_0805_2012Metric_Pad1.15x1.40mm_HandSolder, F.Cu at (199.8, -140.2)
- added D34: LED, LED_SMD:LED_0805_2012Metric_Pad1.15x1.40mm_HandSolder, F.Cu at (203.8, -140.2)
- added D35: LED, LED_SMD:LED_0805_2012Metric_Pad1.15x1.40mm_HandSolder, F.Cu at (207.8, -140.2)
- added D36: LED, LED_SMD:LED_0805_2012Metric_Pad1.15x1.40mm_HandSolder, F.Cu at (211.8, -140.2)
- added D37: LED, LED_SMD:LED_0805_2012Metric_Pad1.15x1.40mm_HandSolder, F.Cu at (215.8, -140.2)
- added D38: LED, LED_SMD:LED_0805_2012Metric_Pad1.15x1.40mm_HandSolder, F.Cu at (219.8, -140.2)
- added D39: LED, LED_SMD:LED_0805_2012Metric_Pad1.15x1.40mm_HandSolder, F.Cu at (223.8, -140.2)
- added D4: LED, LED_SMD:LED_0805_2012Metric_Pad1.15x1.40mm_HandSolder, F.Cu at (84.0, -140.2)
- added D40: LED, LED_SMD:LED_0805_2012Metric_Pad1.15x1.40mm_HandSolder, F.Cu at (227.8, -140.2)
- added D41: LED, LED_SMD:LED_0805_2012Metric_Pad1.15x1.40mm_HandSolder, F.Cu at (231.8, -140.2)
- added D42: LED, LED_SMD:LED_0805_2012Metric_Pad1.15x1.40mm_HandSolder, F.Cu at (235.8, -140.2)
- added D43: LED, LED_SMD:LED_0805_2012Metric_Pad1.15x1.40mm_HandSolder, F.Cu at (239.8, -140.2)
- added D44: LED, LED_SMD:LED_0805_2012Metric_Pad1.15x1.40mm_HandSolder, F.Cu at (243.8, -140.2)
- added D45: LED, LED_SMD:LED_0805_2012Metric_Pad1.15x1.40mm_HandSolder, F.Cu at (247.8, -140.2)
- added D46: LED, LED_SMD:LED_0805_2012Metric_Pad1.15x1.40mm_HandSolder, F.Cu at (251.8, -140.2)
- added D47: LED, LED_SMD:LED_0805_2012Metric_Pad1.15x1.40mm_HandSolder, F.Cu at (255.8, -140.2)
- added D48: LED, LED_SMD:LED_0805_2012Metric_Pad1.15x1.40mm_HandSolder, F.Cu at (259.8, -140.2)
- added D49: LED, LED_SMD:LED_0805_2012Metric_Pad1.15x1.40mm_HandSolder, F.Cu at (263.8, -140.2)
- added D5: LED, LED_SMD:LED_0805_2012Metric_Pad1.15x1.40mm_HandSolder, F.Cu at (88.0, -140.2)
- added D50: LED, LED_SMD:LED_0805_2012Metric_Pad1.15x1.40mm_HandSolder, F.Cu at (267.8, -140.2)
- added D51: LED, LED_SMD:LED_0805_2012Metric_Pad1.15x1.40mm_HandSolder, F.Cu at (271.8, -140.2)
- added D52: LED, LED_SMD:LED_0805_2012Metric_Pad1.15x1.40mm_HandSolder, F.Cu at (275.8, -140.2)
- added D53: LED, LED_SMD:LED_0805_2012Metric_Pad1.15x1.40mm_HandSolder, F.Cu at (279.8, -140.2)
- added D54: LED, LED_SMD:LED_0805_2012Metric_Pad1.15x1.40mm_HandSolder, F.Cu at (283.8, -140.2)
- added D55: LED, LED_SMD:LED_0805_2012Metric_Pad1.15x1.40mm_HandSolder, F.Cu at (287.8, -140.2)
- added D56: LED, LED_SMD:LED_0805_2012Metric_Pad1.15x1.40mm_HandSolder, F.Cu at (291.8, -140.2)
- added D57: LED, LED_SMD:LED_0805_2012Metric_Pad1.15x1.40mm_HandSolder, F.Cu at (295.8, -140.2)
- added D58: LED, LED_SMD:LED_0805_2012Metric_Pad1.15x1.40mm_HandSolder, F.Cu at (299.8, -140.2)
- added D59: LED, LED_SMD:LED_0805_2012Metric_Pad1.15x1.40mm_HandSolder, F.Cu at (303.8, -140.2)
- added D6: LED, LED_SMD:LED_0805_2012Metric_Pad1.15x1.40mm_HandSolder, F.Cu at (92.0, -140.2)
- added D60: LED, LED_SMD:LED_0805_2012Metric_Pad1.15x1.40mm_HandSolder, F.Cu at (307.8, -140.2)
- added D61: LED, LED_SMD:LED_0805_2012Metric_Pad1.15x1.40mm_HandSolder, F.Cu at (311.8, -140.2)
- added D62: LED, LED_SMD:LED_0805_2012Metric_Pad1.15x1.40mm_HandSolder, F.Cu at (315.8, -140.2)
- added D63: LED, LED_SMD:LED_0805_2012Metric_Pad1.15x1.40mm_HandSolder, F.Cu at (319.8, -140.2)
- added D64: LED, LED_SMD:LED_0805_2012Metric_Pad1.15x1.40mm_HandSolder, F.Cu at (323.8, -140.2)
- added D65: LED, LED_SMD:LED_0805_2012Metric_Pad1.15x1.40mm_HandSolder, F.Cu at (60.5, 85.0)
- added D66: LED, LED_SMD:LED_0805_2012Metric_Pad1.15x1.40mm_HandSolder, F.Cu at (51.5, 85.0)
- added D67: LED, LED_SMD:LED_0805_2012Metric_Pad1.15x1.40mm_HandSolder, F.Cu at (56.0, 85.0)
- added D7: LED, LED_SMD:LED_0805_2012Metric_Pad1.15x1.40mm_HandSolder, F.Cu at (96.0, -140.2)
- added D8: LED, LED_SMD:LED_0805_2012Metric_Pad1.15x1.40mm_HandSolder, F.Cu at (100.0, -140.2)
- added D9: LED, LED_SMD:LED_0805_2012Metric_Pad1.15x1.40mm_HandSolder, F.Cu at (104.0, -140.2)
- added JP1: SolderJumper_3_Open, Jumper:SolderJumper-3_P1.3mm_Open_RoundedPad1.0x1.5mm, B.Cu at (247.5, 120.7)
- added JP10: SolderJumper_3_Open, Jumper:SolderJumper-3_P1.3mm_Open_RoundedPad1.0x1.5mm, B.Cu at (61.0, 121.2)
- added JP11: SolderJumper_3_Open, Jumper:SolderJumper-3_P1.3mm_Open_RoundedPad1.0x1.5mm, B.Cu at (149.5, 121.2)
- added JP12: SolderJumper_3_Open, Jumper:SolderJumper-3_P1.3mm_Open_RoundedPad1.0x1.5mm, B.Cu at (152.0, 121.2)
- added JP13: SolderJumper_3_Open, Jumper:SolderJumper-3_P1.3mm_Open_RoundedPad1.0x1.5mm, B.Cu at (154.5, 121.2)
- added JP14: SolderJumper_3_Open, Jumper:SolderJumper-3_P1.3mm_Open_RoundedPad1.0x1.5mm, B.Cu at (157.0, 121.2)
- added JP15: SolderJumper_3_Open, Jumper:SolderJumper-3_P1.3mm_Open_RoundedPad1.0x1.5mm, B.Cu at (159.5, 121.2)
- added JP16: SolderJumper_3_Open, Jumper:SolderJumper-3_P1.3mm_Open_RoundedPad1.0x1.5mm, B.Cu at (261.7, 120.8)
- added JP2: SolderJumper_3_Open, Jumper:SolderJumper-3_P1.3mm_Open_RoundedPad1.0x1.5mm, B.Cu at (250.0, 120.7)
- added JP3: SolderJumper_3_Open, Jumper:SolderJumper-3_P1.3mm_Open_RoundedPad1.0x1.5mm, B.Cu at (252.5, 120.7)
- added JP4: SolderJumper_3_Open, Jumper:SolderJumper-3_P1.3mm_Open_RoundedPad1.0x1.5mm, B.Cu at (255.0, 120.7)
- added JP5: SolderJumper_3_Open, Jumper:SolderJumper-3_P1.3mm_Open_RoundedPad1.0x1.5mm, B.Cu at (257.5, 120.7)
- added JP6: SolderJumper_3_Open, Jumper:SolderJumper-3_P1.3mm_Open_RoundedPad1.0x1.5mm, B.Cu at (51.0, 121.2)
- added JP7: SolderJumper_3_Open, Jumper:SolderJumper-3_P1.3mm_Open_RoundedPad1.0x1.5mm, B.Cu at (53.5, 121.2)
- added JP8: SolderJumper_3_Open, Jumper:SolderJumper-3_P1.3mm_Open_RoundedPad1.0x1.5mm, B.Cu at (56.0, 121.2)
- added JP9: SolderJumper_3_Open, Jumper:SolderJumper-3_P1.3mm_Open_RoundedPad1.0x1.5mm, B.Cu at (58.5, 121.2)
- added R1: 1K, Resistor_SMD:R_0805_2012Metric_Pad1.20x1.40mm_HandSolder, F.Cu at (71.0, -137.2)
- added R10: 1K, Resistor_SMD:R_0805_2012Metric_Pad1.20x1.40mm_HandSolder, F.Cu at (107.0, -137.2)
- added R11: 1K, Resistor_SMD:R_0805_2012Metric_Pad1.20x1.40mm_HandSolder, F.Cu at (111.0, -137.2)
- added R12: 1K, Resistor_SMD:R_0805_2012Metric_Pad1.20x1.40mm_HandSolder, F.Cu at (115.0, -137.2)
- added R13: 1K, Resistor_SMD:R_0805_2012Metric_Pad1.20x1.40mm_HandSolder, F.Cu at (119.0, -137.2)
- added R14: 1K, Resistor_SMD:R_0805_2012Metric_Pad1.20x1.40mm_HandSolder, F.Cu at (123.0, -137.2)
- added R15: 1K, Resistor_SMD:R_0805_2012Metric_Pad1.20x1.40mm_HandSolder, F.Cu at (127.0, -137.2)
- added R16: 1K, Resistor_SMD:R_0805_2012Metric_Pad1.20x1.40mm_HandSolder, F.Cu at (131.0, -137.2)
- added R17: 1K, Resistor_SMD:R_0805_2012Metric_Pad1.20x1.40mm_HandSolder, F.Cu at (135.0, -137.2)
- added R18: 1K, Resistor_SMD:R_0805_2012Metric_Pad1.20x1.40mm_HandSolder, F.Cu at (139.0, -137.2)
- added R19: 1K, Resistor_SMD:R_0805_2012Metric_Pad1.20x1.40mm_HandSolder, F.Cu at (143.0, -137.2)
- added R2: 1K, Resistor_SMD:R_0805_2012Metric_Pad1.20x1.40mm_HandSolder, F.Cu at (75.0, -137.2)
- added R20: 1K, Resistor_SMD:R_0805_2012Metric_Pad1.20x1.40mm_HandSolder, F.Cu at (147.0, -137.2)
- added R21: 1K, Resistor_SMD:R_0805_2012Metric_Pad1.20x1.40mm_HandSolder, F.Cu at (151.0, -137.2)
- added R22: 1K, Resistor_SMD:R_0805_2012Metric_Pad1.20x1.40mm_HandSolder, F.Cu at (155.0, -137.2)
- added R23: 1K, Resistor_SMD:R_0805_2012Metric_Pad1.20x1.40mm_HandSolder, F.Cu at (159.0, -137.2)
- added R24: 1K, Resistor_SMD:R_0805_2012Metric_Pad1.20x1.40mm_HandSolder, F.Cu at (162.9, -137.2)
- added R25: 1K, Resistor_SMD:R_0805_2012Metric_Pad1.20x1.40mm_HandSolder, F.Cu at (166.9, -137.2)
- added R26: 1K, Resistor_SMD:R_0805_2012Metric_Pad1.20x1.40mm_HandSolder, F.Cu at (170.9, -137.2)
- added R27: 1K, Resistor_SMD:R_0805_2012Metric_Pad1.20x1.40mm_HandSolder, F.Cu at (174.9, -137.2)
- added R28: 1K, Resistor_SMD:R_0805_2012Metric_Pad1.20x1.40mm_HandSolder, F.Cu at (178.9, -137.2)
- added R29: 1K, Resistor_SMD:R_0805_2012Metric_Pad1.20x1.40mm_HandSolder, F.Cu at (182.9, -137.2)
- added R3: 1K, Resistor_SMD:R_0805_2012Metric_Pad1.20x1.40mm_HandSolder, F.Cu at (79.0, -137.2)
- added R30: 1K, Resistor_SMD:R_0805_2012Metric_Pad1.20x1.40mm_HandSolder, F.Cu at (186.9, -137.2)
- added R31: 1K, Resistor_SMD:R_0805_2012Metric_Pad1.20x1.40mm_HandSolder, F.Cu at (190.8, -137.2)
- added R32: 1K, Resistor_SMD:R_0805_2012Metric_Pad1.20x1.40mm_HandSolder, F.Cu at (194.8, -137.2)
- added R33: 1K, Resistor_SMD:R_0805_2012Metric_Pad1.20x1.40mm_HandSolder, F.Cu at (198.8, -137.2)
- added R34: 1K, Resistor_SMD:R_0805_2012Metric_Pad1.20x1.40mm_HandSolder, F.Cu at (202.8, -137.2)
- added R35: 1K, Resistor_SMD:R_0805_2012Metric_Pad1.20x1.40mm_HandSolder, F.Cu at (206.8, -137.2)
- added R36: 1K, Resistor_SMD:R_0805_2012Metric_Pad1.20x1.40mm_HandSolder, F.Cu at (210.8, -137.2)
- added R37: 1K, Resistor_SMD:R_0805_2012Metric_Pad1.20x1.40mm_HandSolder, F.Cu at (214.8, -137.2)
- added R38: 1K, Resistor_SMD:R_0805_2012Metric_Pad1.20x1.40mm_HandSolder, F.Cu at (218.8, -137.2)
- added R39: 1K, Resistor_SMD:R_0805_2012Metric_Pad1.20x1.40mm_HandSolder, F.Cu at (222.8, -137.2)
- added R4: 1K, Resistor_SMD:R_0805_2012Metric_Pad1.20x1.40mm_HandSolder, F.Cu at (83.0, -137.2)
- added R40: 1K, Resistor_SMD:R_0805_2012Metric_Pad1.20x1.40mm_HandSolder, F.Cu at (226.8, -137.2)
- added R41: 1K, Resistor_SMD:R_0805_2012Metric_Pad1.20x1.40mm_HandSolder, F.Cu at (230.8, -137.2)
- added R42: 1K, Resistor_SMD:R_0805_2012Metric_Pad1.20x1.40mm_HandSolder, F.Cu at (234.8, -137.2)
- added R43: 1K, Resistor_SMD:R_0805_2012Metric_Pad1.20x1.40mm_HandSolder, F.Cu at (238.8, -137.2)
- added R44: 1K, Resistor_SMD:R_0805_2012Metric_Pad1.20x1.40mm_HandSolder, F.Cu at (242.8, -137.2)
- added R45: 1K, Resistor_SMD:R_0805_2012Metric_Pad1.20x1.40mm_HandSolder, F.Cu at (246.8, -137.2)
- added R46: 1K, Resistor_SMD:R_0805_2012Metric_Pad1.20x1.40mm_HandSolder, F.Cu at (250.8, -137.2)
- added R47: 1K, Resistor_SMD:R_0805_2012Metric_Pad1.20x1.40mm_HandSolder, F.Cu at (254.8, -137.2)
- added R48: 1K, Resistor_SMD:R_0805_2012Metric_Pad1.20x1.40mm_HandSolder, F.Cu at (258.8, -137.2)
- added R49: 1K, Resistor_SMD:R_0805_2012Metric_Pad1.20x1.40mm_HandSolder, F.Cu at (262.8, -137.2)
- added R5: 1K, Resistor_SMD:R_0805_2012Metric_Pad1.20x1.40mm_HandSolder, F.Cu at (87.0, -137.2)
- added R50: 1K, Resistor_SMD:R_0805_2012Metric_Pad1.20x1.40mm_HandSolder, F.Cu at (266.8, -137.2)
- added R51: 1K, Resistor_SMD:R_0805_2012Metric_Pad1.20x1.40mm_HandSolder, F.Cu at (270.8, -137.2)
- added R52: 1K, Resistor_SMD:R_0805_2012Metric_Pad1.20x1.40mm_HandSolder, F.Cu at (274.8, -137.2)
- added R53: 1K, Resistor_SMD:R_0805_2012Metric_Pad1.20x1.40mm_HandSolder, F.Cu at (278.8, -137.2)
- added R54: 1K, Resistor_SMD:R_0805_2012Metric_Pad1.20x1.40mm_HandSolder, F.Cu at (282.8, -137.2)
- added R55: 1K, Resistor_SMD:R_0805_2012Metric_Pad1.20x1.40mm_HandSolder, F.Cu at (286.6, -137.2)
- added R56: 1K, Resistor_SMD:R_0805_2012Metric_Pad1.20x1.40mm_HandSolder, F.Cu at (290.8, -137.2)
- added R57: 1K, Resistor_SMD:R_0805_2012Metric_Pad1.20x1.40mm_HandSolder, F.Cu at (294.8, -137.2)
- added R58: 1K, Resistor_SMD:R_0805_2012Metric_Pad1.20x1.40mm_HandSolder, F.Cu at (298.8, -137.2)
- added R59: 1K, Resistor_SMD:R_0805_2012Metric_Pad1.20x1.40mm_HandSolder, F.Cu at (302.8, -137.2)
- added R6: 1K, Resistor_SMD:R_0805_2012Metric_Pad1.20x1.40mm_HandSolder, F.Cu at (91.0, -137.2)
- added R60: 1K, Resistor_SMD:R_0805_2012Metric_Pad1.20x1.40mm_HandSolder, F.Cu at (306.8, -137.2)
- added R61: 1K, Resistor_SMD:R_0805_2012Metric_Pad1.20x1.40mm_HandSolder, F.Cu at (310.8, -137.2)
- added R62: 1K, Resistor_SMD:R_0805_2012Metric_Pad1.20x1.40mm_HandSolder, F.Cu at (314.8, -137.2)
- added R63: 1K, Resistor_SMD:R_0805_2012Metric_Pad1.20x1.40mm_HandSolder, F.Cu at (318.8, -137.2)
- added R64: 1K, Resistor_SMD:R_0805_2012Metric_Pad1.20x1.40mm_HandSolder, F.Cu at (322.8, -137.2)
- added R65: 1K, Resistor_SMD:R_0805_2012Metric_Pad1.20x1.40mm_HandSolder, B.Cu at (57.0, 69.1)
- added R66: 1K, Resistor_SMD:R_0805_2012Metric_Pad1.20x1.40mm_HandSolder, B.Cu at (57.0, 72.0)
- added R67: 1K, Resistor_SMD:R_0805_2012Metric_Pad1.20x1.40mm_HandSolder, B.Cu at (57.0, 75.0)
- added R7: 1K, Resistor_SMD:R_0805_2012Metric_Pad1.20x1.40mm_HandSolder, F.Cu at (95.0, -137.2)
- added R8: 1K, Resistor_SMD:R_0805_2012Metric_Pad1.20x1.40mm_HandSolder, F.Cu at (99.0, -137.2)
- added R9: 1K, Resistor_SMD:R_0805_2012Metric_Pad1.20x1.40mm_HandSolder, F.Cu at (103.0, -137.2)
- added U1: 74LS00, Package_SO:SOIC-14_3.9x8.7mm_P1.27mm, B.Cu at (247.0, 112.5)
- added U10: 74LS273, Package_SO:SOIC-20W_7.5x12.8mm_P1.27mm, B.Cu at (310.5, 114.0)
- added U11: 74LS273, Package_SO:SOIC-20W_7.5x12.8mm_P1.27mm, B.Cu at (325.5, 114.0)
- added U12: 74LS541, Package_SO:SOIC-20W_7.5x12.8mm_P1.27mm, F.Cu at (72.4, 113.7)
- added U13: 74LS541, Package_SO:SOIC-20W_7.5x12.8mm_P1.27mm, B.Cu at (88.4, 164.6)
- added U14: 74LS541, Package_SO:SOIC-20W_7.5x12.8mm_P1.27mm, B.Cu at (106.1, 150.3)
- added U15: 74LS541, Package_SO:SOIC-20W_7.5x12.8mm_P1.27mm, B.Cu at (122.8, 153.8)
- added U16: 74LS541, Package_SO:SOIC-20W_7.5x12.8mm_P1.27mm, B.Cu at (73.6, 116.9)
- added U17: 74LS541, Package_SO:SOIC-20W_7.5x12.8mm_P1.27mm, B.Cu at (91.3, 116.8)
- added U18: 74LS541, Package_SO:SOIC-20W_7.5x12.8mm_P1.27mm, B.Cu at (108.4, 116.8)
- added U19: 74LS541, Package_SO:SOIC-20W_7.5x12.8mm_P1.27mm, B.Cu at (124.3, 117.2)
- added U2: 74LS00, Package_SO:SOIC-14_3.9x8.7mm_P1.27mm, B.Cu at (258.2, 112.5)
- added U20: 74LS04, Package_SO:SOIC-14_3.9x8.7mm_P1.27mm, B.Cu at (56.0, 113.5)
- added U21: 74LS30, Package_SO:SOIC-14_3.9x8.7mm_P1.27mm, B.Cu at (55.7, 104.0)
- added U22: 74LS541, Package_SO:SOIC-20W_7.5x12.8mm_P1.27mm, B.Cu at (170.5, 149.8)
- added U23: 74LS541, Package_SO:SOIC-20W_7.5x12.8mm_P1.27mm, B.Cu at (188.5, 150.0)
- added U24: 74LS541, Package_SO:SOIC-20W_7.5x12.8mm_P1.27mm, B.Cu at (205.0, 150.0)
- added U25: 74LS541, Package_SO:SOIC-20W_7.5x12.8mm_P1.27mm, B.Cu at (223.8, 150.3)
- added U26: 74LS541, Package_SO:SOIC-20W_7.5x12.8mm_P1.27mm, B.Cu at (174.0, 112.0)
- added U27: 74LS541, Package_SO:SOIC-20W_7.5x12.8mm_P1.27mm, B.Cu at (191.5, 112.0)
- added U28: 74LS541, Package_SO:SOIC-20W_7.5x12.8mm_P1.27mm, B.Cu at (209.1, 111.8)
- added U29: 74LS541, Package_SO:SOIC-20W_7.5x12.8mm_P1.27mm, B.Cu at (225.6, 111.8)
- added U3: 74LS30, Package_SO:SOIC-14_3.9x8.7mm_P1.27mm, B.Cu at (253.0, 102.5)
- added U30: 74LS04, Package_SO:SOIC-14_3.9x8.7mm_P1.27mm, B.Cu at (154.0, 112.0)
- added U31: 74LS30, Package_SO:SOIC-14_3.9x8.7mm_P1.27mm, B.Cu at (142.1, 112.8)
- added U4: 74LS273, Package_SO:SOIC-20W_7.5x12.8mm_P1.27mm, F.Cu at (274.6, 115.3)
- added U5: 74LS273, Package_SO:SOIC-20W_7.5x12.8mm_P1.27mm, F.Cu at (291.4, 115.8)
- added U6: 74LS273, Package_SO:SOIC-20W_7.5x12.8mm_P1.27mm, F.Cu at (310.6, 114.1)
- added U7: 74LS273, Package_SO:SOIC-20W_7.5x12.8mm_P1.27mm, F.Cu at (325.4, 114.6)
- added U8: 74LS273, Package_SO:SOIC-20W_7.5x12.8mm_P1.27mm, B.Cu at (274.4, 116.3)
- added U9: 74LS273, Package_SO:SOIC-20W_7.5x12.8mm_P1.27mm, B.Cu at (291.0, 115.5)
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Connections:
- J1 pad A10: Net-(J1-+3.3V-PadA10) -> +3V3
- J1 pad A11: unconnected-(J1-~{PERST}-PadA11) -> ~{RST}
- J1 pad A13: unconnected-(J1-REFCLK+-PadA13) -> CLK_PH0
- J1 pad A14: unconnected-(J1-REFCLK--PadA14) -> CLK_PH1
- J1 pad A16: read_a32 -> write32
- J1 pad A17: read_a33 -> write33
- J1 pad A2: Net-(J1-+12V-PadA2) -> unconnected-(J1-+12V-PadA2)_1
- J1 pad A21: read_a34 -> write34
- J1 pad A22: read_a35 -> write35
- J1 pad A25: read_a36 -> write36
- J1 pad A26: read_a37 -> write37
- J1 pad A29: read_a38 -> write38
- J1 pad A3: Net-(J1-+12V-PadA2) -> unconnected-(J1-+12V-PadA2)_3
- J1 pad A30: read_a39 -> write39
- J1 pad A35: read_a40 -> write40
- J1 pad A36: read_a41 -> write41
- J1 pad A39: read_a42 -> write42
- J1 pad A40: read_a43 -> write43
- J1 pad A43: read_a44 -> write44
- J1 pad A44: read_a45 -> write45
- J1 pad A47: read_a46 -> write46
- J1 pad A48: read_a47 -> write47
- J1 pad A5: unconnected-(J1-JTAG2-PadA5) -> /Write In/write_sel1
- J1 pad A52: read_a48 -> write48
- J1 pad A53: read_a49 -> write49
- J1 pad A56: read_a50 -> write50
- J1 pad A57: read_a51 -> write51
- J1 pad A6: unconnected-(J1-JTAG3-PadA6) -> /Write In/write_sel2
- J1 pad A60: read_a52 -> write52
- J1 pad A61: read_a53 -> write53
- J1 pad A64: read_a54 -> write54
- J1 pad A65: read_a55 -> write55
- J1 pad A68: read_a56 -> write56
- J1 pad A69: read_a57 -> write57
- J1 pad A7: unconnected-(J1-JTAG4-PadA7) -> /Write In/write_sel3
- J1 pad A72: read_a58 -> write58
- J1 pad A73: read_a59 -> write59
- J1 pad A76: read_a60 -> write60
- J1 pad A77: read_a61 -> write61
- J1 pad A8: unconnected-(J1-JTAG5-PadA8) -> /Write In/write_sel4
- J1 pad A80: read_a62 -> write62
- J1 pad A81: read_a63 -> write63
- J1 pad A9: Net-(J1-+3.3V-PadA10) -> +3V3
- J1 pad B1: Net-(J1-+12V-PadA2) -> unconnected-(J1-+12V-PadA2)
- J1 pad B14: /read_a00 -> write0
- J1 pad B15: /read_a01 -> write1
- J1 pad B19: /read_a02 -> write2
- J1 pad B2: Net-(J1-+12V-PadA2) -> unconnected-(J1-+12V-PadA2)_2
- J1 pad B20: /read_a03 -> write3
- J1 pad B23: /read_a04 -> write4
- J1 pad B24: /read_a05 -> write5
- J1 pad B27: /read_a06 -> write6
- J1 pad B28: /read_a07 -> write7
- J1 pad B3: Net-(J1-+12V-PadA2) -> unconnected-(J1-+12V-PadA2)_4
- J1 pad B33: /read_a08 -> write8
- J1 pad B34: /read_a09 -> write9
- J1 pad B37: read_a10 -> write10
- J1 pad B38: read_a11 -> write11
- J1 pad B41: read_a12 -> write12
- J1 pad B42: read_a13 -> write13
- J1 pad B45: read_a14 -> write14
- J1 pad B46: read_a15 -> write15
- J1 pad B50: read_a16 -> write16
- J1 pad B51: read_a17 -> write17
- J1 pad B54: read_a18 -> write18
- J1 pad B55: read_a19 -> write19
- J1 pad B58: read_a20 -> write20
- J1 pad B59: read_a21 -> write21
- J1 pad B62: read_a22 -> write22
- J1 pad B63: read_a23 -> write23
- J1 pad B66: read_a24 -> write24
- J1 pad B67: read_a25 -> write25
- J1 pad B70: read_a26 -> write26
- J1 pad B71: read_a27 -> write27
- J1 pad B74: read_a28 -> write28
- J1 pad B75: read_a29 -> write29
- J1 pad B78: read_a30 -> write30
- J1 pad B79: read_a31 -> write31
- J1 pad B8: Net-(J1-+3.3V-PadA10) -> +3V3
- J1 pad B9: unconnected-(J1-JTAG1-PadB9) -> /Write In/write_sel0
- J2 pad A10: Net-(J2-+3.3V-PadA10) -> +3V3
- J2 pad A16: read_b32 -> read_a32
- J2 pad A17: read_b33 -> read_a33
- J2 pad A2: Net-(J2-+12V-PadA2) -> unconnected-(J2-+12V-PadA2)_3
- J2 pad A21: read_b34 -> read_a34
- J2 pad A22: read_b35 -> read_a35
- J2 pad A25: read_b36 -> read_a36
- J2 pad A26: read_b37 -> read_a37
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Routing:
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Other:
- copper layers 2 -> 4

Commit message: More routing done.
Parts:
- moved D1 201.4 mm to (79.1, 61.1)
- moved D10 201.4 mm to (115.1, 61.1)
- moved D11 201.4 mm to (119.1, 61.1)
- moved D12 201.4 mm to (123.1, 61.1)
- moved D13 201.4 mm to (127.1, 61.1)
- moved D14 201.4 mm to (131.1, 61.1)
- moved D15 201.4 mm to (135.1, 61.1)
- moved D16 201.4 mm to (139.1, 61.1)
- moved D17 201.4 mm to (143.1, 61.1)
- moved D18 201.4 mm to (147.1, 61.1)
- moved D19 201.4 mm to (151.1, 61.1)
- moved D2 201.4 mm to (83.1, 61.1)
- moved D20 201.4 mm to (155.1, 61.1)
- moved D21 201.4 mm to (159.1, 61.1)
- moved D22 201.4 mm to (163.1, 61.1)
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Routing:
- net latched33: track 0.00 -> 309.0 mm
- net latched34: track 0.00 -> 307.9 mm
- net latched36: track 10.2 -> 305.7 mm
- net latched37: track 10.0 -> 304.6 mm
- net latched35: track 12.3 -> 306.8 mm
- net latched38: track 11.0 -> 303.6 mm
- net latched39: track 11.9 -> 302.4 mm
- net latched32: track 25.0 -> 310.2 mm
- net latched41: track 7.00 -> 292.1 mm
- net latched40: track 9.50 -> 293.2 mm
- net latched42: track 8.50 -> 291.0 mm
- net latched43: track 9.40 -> 289.9 mm
- net latched44: track 9.70 -> 288.7 mm
- net latched45: track 12.1 -> 287.6 mm
- net latched47: track 13.3 -> 285.4 mm
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Other:
- board size 284.3 x 41.5 mm -> 284.6 x 65.8 mm

Commit message: Read A Port mostly routed.
Parts:
- U13, U14, U15: moved to F.Cu
- moved U13 47.7 mm to (90.7, 117.0)
- moved U12 41.7 mm to (73.6, 116.9)
- moved U15 36.9 mm to (125.2, 117.0)
- moved U14 33.4 mm to (108.0, 117.0)
Connections:
- U12 pad 11: read_a7 -> read_a0
- U12 pad 12: read_a6 -> read_a1
- U12 pad 13: read_a5 -> read_a2
- U12 pad 14: read_a4 -> read_a3
- U12 pad 15: read_a3 -> read_a4
- U12 pad 16: read_a2 -> read_a5
- U12 pad 17: read_a1 -> read_a6
- U12 pad 18: read_a0 -> read_a7
- U12 pad 2: latched0 -> latched7
- U12 pad 3: latched1 -> latched6
- U12 pad 4: latched2 -> latched5
- U12 pad 5: latched3 -> latched4
- U12 pad 6: latched4 -> latched3
- U12 pad 7: latched5 -> latched2
- U12 pad 8: latched6 -> latched1
- U12 pad 9: latched7 -> latched0
- U13 pad 11: read_a15 -> read_a8
- U13 pad 12: read_a14 -> read_a9
- U13 pad 13: read_a13 -> read_a10
- U13 pad 14: read_a12 -> read_a11
- U13 pad 15: read_a11 -> read_a12
- U13 pad 16: read_a10 -> read_a13
- U13 pad 17: read_a9 -> read_a14
- U13 pad 18: read_a8 -> read_a15
- U13 pad 2: latched8 -> latched15
- U13 pad 3: latched9 -> latched14
- U13 pad 4: latched10 -> latched13
- U13 pad 5: latched11 -> latched12
- U13 pad 6: latched12 -> latched11
- U13 pad 7: latched13 -> latched10
- U13 pad 8: latched14 -> latched9
- U13 pad 9: latched15 -> latched8
- U14 pad 11: read_a23 -> read_a16
- U14 pad 12: read_a22 -> read_a17
- U14 pad 13: read_a21 -> read_a18
- U14 pad 14: read_a20 -> read_a19
- U14 pad 15: read_a19 -> read_a20
- U14 pad 16: read_a18 -> read_a21
- U14 pad 17: read_a17 -> read_a22
- U14 pad 18: read_a16 -> read_a23
- U14 pad 2: latched16 -> latched23
- U14 pad 3: latched17 -> latched22
- U14 pad 4: latched18 -> latched21
- U14 pad 5: latched19 -> latched20
- U14 pad 6: latched20 -> latched19
- U14 pad 7: latched21 -> latched18
- U14 pad 8: latched22 -> latched17
- U14 pad 9: latched23 -> latched16
- U15 pad 11: read_a31 -> read_a24
- U15 pad 12: read_a30 -> read_a25
- U15 pad 13: read_a29 -> read_a26
- U15 pad 14: read_a28 -> read_a27
- U15 pad 15: read_a27 -> read_a28
- U15 pad 16: read_a26 -> read_a29
- U15 pad 17: read_a25 -> read_a30
- U15 pad 18: read_a24 -> read_a31
- U15 pad 2: latched24 -> latched31
- U15 pad 3: latched25 -> latched30
- U15 pad 4: latched26 -> latched29
- U15 pad 5: latched27 -> latched28
- U15 pad 6: latched28 -> latched27
- U15 pad 7: latched29 -> latched26
- U15 pad 8: latched30 -> latched25
- U15 pad 9: latched31 -> latched24
Routing:
- net latched0: track 261.1 -> 310.1 mm, vias 1 -> 2
- net latched1: track 261.8 -> 309.1 mm, vias 1 -> 2
- net latched2: track 262.3 -> 307.9 mm, vias 1 -> 2
- net latched3: track 262.9 -> 306.8 mm, vias 1 -> 2
- net latched4: track 263.5 -> 305.7 mm, vias 1 -> 2
- net latched5: track 264.1 -> 304.6 mm, vias 1 -> 2
- net latched6: track 264.7 -> 303.4 mm, vias 1 -> 2
- net latched7: track 265.3 -> 302.3 mm, vias 1 -> 2
- net latched31: track 279.9 -> 252.0 mm, vias 1 -> 2
- net latched8: track 265.9 -> 293.1 mm, vias 1 -> 2
- net latched30: track 279.2 -> 253.0 mm, vias 1 -> 2
- net latched9: track 266.5 -> 292.0 mm, vias 1 -> 2
- net latched29: track 278.5 -> 254.1 mm, vias 1 -> 2
- net latched10: track 267.1 -> 290.9 mm, vias 1 -> 2
- net latched28: track 277.9 -> 255.1 mm, vias 1 -> 2
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Other:
- board size 284.6 x 65.8 mm -> 284.3 x 65.8 mm

Commit message: Getting close to done with Read A Port.
Parts:
- C12, C13, C14, C15, C21, R65, R66, R67, U21: moved to F.Cu
- moved C15 141.1 mm to (133.8, 121.5), turned to 90 degrees
- moved C19 129.9 mm to (116.6, 121.3), turned to 90 degrees
- moved C14 125.2 mm to (116.6, 121.4), turned to 90 degrees
- moved C18 114.4 mm to (99.4, 121.3), turned to 90 degrees
- moved C13 109.9 mm to (99.4, 121.4), turned to 90 degrees
- moved C17 99.5 mm to (82.1, 121.4), turned to 90 degrees
- moved C12 95.1 mm to (82.1, 121.3), turned to 90 degrees
- moved C16 71.9 mm to (64.2, 116.0), turned to 90 degrees
- moved D65 71.7 mm to (33.0, 82.8)
- moved D66 71.7 mm to (24.0, 82.8)
- moved D67 71.7 mm to (28.5, 82.8)
- moved R67 71.7 mm to (29.4, 72.8), turned to 0 degrees
- moved R65 71.7 mm to (29.4, 66.9), turned to 0 degrees
- moved R66 71.7 mm to (29.4, 69.8), turned to 0 degrees
- moved C20 63.4 mm to (41.1, 128.6)
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Connections:
- U20 pad 10: Net-(JP10-B) -> Net-(JP9-B)
- U20 pad 11: /Read Out A/read_a_sel4 -> /Read Out A/read_a_sel3
- U20 pad 12: read_a_en -> Net-(JP8-B)
- U20 pad 13: ~{read_a_en} -> /Read Out A/read_a_sel2
- U20 pad 5: /Read Out A/read_a_sel2 -> ~{read_a_en}
- U20 pad 6: Net-(JP8-B) -> read_a_en
- U20 pad 8: Net-(JP9-B) -> Net-(JP10-B)
- U20 pad 9: /Read Out A/read_a_sel3 -> /Read Out A/read_a_sel4
Routing:
- net ~{read_a_en}: track 0.00 -> 102.9 mm, vias 0 -> 6
- net GND: track 348.0 -> 417.9 mm, vias 99 -> 116
- net +3V3: track 10.9 -> 64.2 mm, vias 2 -> 12
- net read_a_en: track 0.00 -> 47.3 mm
- net Net-(JP10-C): track 0.00 -> 13.8 mm, vias 0 -> 1
- net Net-(JP9-C): track 0.00 -> 12.0 mm, vias 0 -> 1
- net Net-(JP8-C): track 0.00 -> 10.9 mm, vias 0 -> 1
- net Net-(JP7-B): track 0.00 -> 10.8 mm
- net Net-(JP7-C): track 0.00 -> 10.1 mm, vias 0 -> 1
- net Net-(JP6-B): track 0.00 -> 10.1 mm
- net Net-(JP6-C): track 0.00 -> 9.36 mm, vias 0 -> 1
- net /Read Out A/read_a_sel1: track 7.71 -> 15.2 mm
- net Net-(JP10-B): track 0.00 -> 6.83 mm
- net Net-(JP9-B): track 0.00 -> 5.81 mm
- net Net-(JP8-B): track 0.00 -> 5.02 mm
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
Commit message: Progress on Read B Port.
Parts:
- C20, C22, C23, C24, C25, U22, U23, U24, U25: moved to F.Cu
- moved D65 35.7 mm to (61.4, 61.2)
- moved D67 35.4 mm to (56.6, 61.2)
- moved D66 35.3 mm to (51.9, 61.2)
- moved U25 33.3 mm to (224.9, 117.1)
- moved U24 33.1 mm to (208.1, 117.0)
- moved U23 33.0 mm to (190.7, 117.1)
- moved U22 32.9 mm to (173.3, 117.1)
- moved R65 31.1 mm to (60.4, 64.2), turned to -90 degrees
- moved R67 27.4 mm to (55.5, 64.2), turned to -90 degrees
- moved C20 22.2 mm to (50.5, 108.4), turned to -90 degrees
- moved R66 22.2 mm to (50.9, 64.2), turned to -90 degrees
- moved C21 19.7 mm to (62.0, 114.4), turned to -90 degrees
- moved C22 17.5 mm to (171.7, 160.9), turned to 0 degrees
- moved C23 17.5 mm to (171.7, 163.9), turned to 0 degrees
- moved C24 17.5 mm to (171.7, 166.9), turned to 0 degrees
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Connections:
- U22 pad 11: read_b7 -> read_b0
- U22 pad 12: read_b6 -> read_b1
- U22 pad 13: read_b5 -> read_b2
- U22 pad 14: read_b4 -> read_b3
- U22 pad 15: read_b3 -> read_b4
- U22 pad 16: read_b2 -> read_b5
- U22 pad 17: read_b1 -> read_b6
- U22 pad 18: read_b0 -> read_b7
- U22 pad 2: latched0 -> latched7
- U22 pad 3: latched1 -> latched6
- U22 pad 4: latched2 -> latched5
- U22 pad 5: latched3 -> latched4
- U22 pad 6: latched4 -> latched3
- U22 pad 7: latched5 -> latched2
- U22 pad 8: latched6 -> latched1
- U22 pad 9: latched7 -> latched0
- U23 pad 11: read_b15 -> read_b8
- U23 pad 12: read_b14 -> read_b9
- U23 pad 13: read_b13 -> read_b10
- U23 pad 14: read_b12 -> read_b11
- U23 pad 15: read_b11 -> read_b12
- U23 pad 16: read_b10 -> read_b13
- U23 pad 17: read_b9 -> read_b14
- U23 pad 18: read_b8 -> read_b15
- U23 pad 2: latched8 -> latched15
- U23 pad 3: latched9 -> latched14
- U23 pad 4: latched10 -> latched13
- U23 pad 5: latched11 -> latched12
- U23 pad 6: latched12 -> latched11
- U23 pad 7: latched13 -> latched10
- U23 pad 8: latched14 -> latched9
- U23 pad 9: latched15 -> latched8
- U24 pad 11: read_b23 -> read_b16
- U24 pad 12: read_b22 -> read_b17
- U24 pad 13: read_b21 -> read_b18
- U24 pad 14: read_b20 -> read_b19
- U24 pad 15: read_b19 -> read_b20
- U24 pad 16: read_b18 -> read_b21
- U24 pad 17: read_b17 -> read_b22
- U24 pad 18: read_b16 -> read_b23
- U24 pad 2: latched16 -> latched23
- U24 pad 3: latched17 -> latched22
- U24 pad 4: latched18 -> latched21
- U24 pad 5: latched19 -> latched20
- U24 pad 6: latched20 -> latched19
- U24 pad 7: latched21 -> latched18
- U24 pad 8: latched22 -> latched17
- U24 pad 9: latched23 -> latched16
- U25 pad 11: read_b31 -> read_b24
- U25 pad 12: read_b30 -> read_b25
- U25 pad 13: read_b29 -> read_b26
- U25 pad 14: read_b28 -> read_b27
- U25 pad 15: read_b27 -> read_b28
- U25 pad 16: read_b26 -> read_b29
- U25 pad 17: read_b25 -> read_b30
- U25 pad 18: read_b24 -> read_b31
- U25 pad 2: latched24 -> latched31
- U25 pad 3: latched25 -> latched30
- U25 pad 4: latched26 -> latched29
- U25 pad 5: latched27 -> latched28
- U25 pad 6: latched28 -> latched27
- U25 pad 7: latched29 -> latched26
- U25 pad 8: latched30 -> latched25
- U25 pad 9: latched31 -> latched24
Routing:
- net GND: track 417.9 -> 667.4 mm, vias 116 -> 155
- net latched0: track 310.1 -> 356.0 mm, vias 2 -> 3
- net latched1: track 309.1 -> 354.3 mm, vias 2 -> 3
- net latched2: track 307.9 -> 352.6 mm, vias 2 -> 3
- net latched3: track 306.8 -> 350.9 mm, vias 2 -> 3
- net latched4: track 305.7 -> 349.1 mm, vias 2 -> 3
- net latched5: track 304.6 -> 347.4 mm, vias 2 -> 3
- net latched6: track 303.4 -> 345.8 mm, vias 2 -> 3
- net latched7: track 302.3 -> 344.0 mm, vias 2 -> 3
- net latched8: track 293.1 -> 334.2 mm, vias 2 -> 3
- net latched9: track 292.0 -> 332.5 mm, vias 2 -> 3
- net latched10: track 290.9 -> 330.8 mm, vias 2 -> 3
- net latched11: track 289.8 -> 329.1 mm, vias 2 -> 3
- net latched12: track 288.7 -> 327.4 mm, vias 2 -> 3
- net latched13: track 287.6 -> 325.7 mm, vias 2 -> 3
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Other:
- board text added: "READ A"

Commit message: Moar progress.  Working on the write in latch.
Parts:
- C4, C5, C6, C7: moved to F.Cu
- moved C8 70.7 mm to (273.3, 109.0), turned to 0 degrees
- moved C4 67.6 mm to (275.4, 109.0)
- moved C9 54.7 mm to (290.4, 109.1), turned to 0 degrees
- moved C5 50.6 mm to (292.5, 109.1)
- moved C10 39.7 mm to (307.6, 109.0), turned to 0 degrees
- moved C6 33.9 mm to (309.7, 109.0)
- moved C11 28.1 mm to (324.5, 109.0), turned to 0 degrees
- moved C7 18.9 mm to (326.5, 109.0)
- moved U6 3.38 mm to (308.6, 116.8)
- moved U10 3.34 mm to (308.6, 116.8)
- moved U11 2.83 mm to (325.5, 116.8)
- moved U7 2.25 mm to (325.5, 116.8)
- moved U4 1.51 mm to (274.4, 116.8)
- moved U9 1.46 mm to (291.6, 116.9)
- moved U5 1.05 mm to (291.6, 116.9)
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Connections:
- U10 pad 12: latched52 -> latched48
- U10 pad 13: write52 -> write48
- U10 pad 14: write53 -> write49
- U10 pad 15: latched53 -> latched49
- U10 pad 16: latched54 -> latched50
- U10 pad 17: write54 -> write50
- U10 pad 18: write55 -> write51
- U10 pad 19: latched55 -> latched51
- U10 pad 2: latched48 -> latched52
- U10 pad 3: write48 -> write52
- U10 pad 4: write49 -> write53
- U10 pad 5: latched49 -> latched53
- U10 pad 6: latched50 -> latched54
- U10 pad 7: write50 -> write54
- U10 pad 8: write51 -> write55
- U10 pad 9: latched51 -> latched55
- U11 pad 12: latched60 -> latched56
- U11 pad 13: write60 -> write56
- U11 pad 14: write61 -> write57
- U11 pad 15: latched61 -> latched57
- U11 pad 16: latched62 -> latched58
- U11 pad 17: write62 -> write58
- U11 pad 18: write63 -> write59
- U11 pad 19: latched63 -> latched59
- U11 pad 2: latched56 -> latched60
- U11 pad 3: write56 -> write60
- U11 pad 4: write57 -> write61
- U11 pad 5: latched57 -> latched61
- U11 pad 6: latched58 -> latched62
- U11 pad 7: write58 -> write62
- U11 pad 8: write59 -> write63
- U11 pad 9: latched59 -> latched63
- U4 pad 12: latched4 -> latched7
- U4 pad 13: write4 -> write7
- U4 pad 14: write5 -> write6
- U4 pad 15: latched5 -> latched6
- U4 pad 16: latched6 -> latched5
- U4 pad 17: write6 -> write5
- U4 pad 18: write7 -> write4
- U4 pad 19: latched7 -> latched4
- U4 pad 2: latched0 -> latched3
- U4 pad 3: write0 -> write3
- U4 pad 4: write1 -> write2
- U4 pad 5: latched1 -> latched2
- U4 pad 6: latched2 -> latched1
- U4 pad 7: write2 -> write1
- U4 pad 8: write3 -> write0
- U4 pad 9: latched3 -> latched0
- U5 pad 12: latched12 -> latched15
- U5 pad 13: write12 -> write15
- U5 pad 14: write13 -> write14
- U5 pad 15: latched13 -> latched14
- U5 pad 16: latched14 -> latched13
- U5 pad 17: write14 -> write13
- U5 pad 18: write15 -> write12
- U5 pad 19: latched15 -> latched12
- U5 pad 2: latched8 -> latched11
- U5 pad 3: write8 -> write11
- U5 pad 4: write9 -> write10
- U5 pad 5: latched9 -> latched10
- U5 pad 6: latched10 -> latched9
- U5 pad 7: write10 -> write9
- U5 pad 8: write11 -> write8
- U5 pad 9: latched11 -> latched8
- U6 pad 12: latched20 -> latched23
- U6 pad 13: write20 -> write23
- U6 pad 14: write21 -> write22
- U6 pad 15: latched21 -> latched22
- U6 pad 16: latched22 -> latched21
- U6 pad 17: write22 -> write21
- U6 pad 18: write23 -> write20
- U6 pad 19: latched23 -> latched20
- U6 pad 2: latched16 -> latched19
- U6 pad 3: write16 -> write19
- U6 pad 4: write17 -> write18
- U6 pad 5: latched17 -> latched18
- U6 pad 6: latched18 -> latched17
- U6 pad 7: write18 -> write17
- U6 pad 8: write19 -> write16
- U6 pad 9: latched19 -> latched16
- U7 pad 12: latched28 -> latched31
- U7 pad 13: write28 -> write31
- U7 pad 14: write29 -> write30
- U7 pad 15: latched29 -> latched30
- U7 pad 16: latched30 -> latched29
- U7 pad 17: write30 -> write29
- U7 pad 18: write31 -> write28
- U7 pad 19: latched31 -> latched28
- U7 pad 2: latched24 -> latched27
- U7 pad 3: write24 -> write27
- U7 pad 4: write25 -> write26
- U7 pad 5: latched25 -> latched26
- U7 pad 6: latched26 -> latched25
- U7 pad 7: write26 -> write25
- U7 pad 8: write27 -> write24
- U7 pad 9: latched27 -> latched24
- U8 pad 12: latched36 -> latched32
- U8 pad 13: write36 -> write32
- U8 pad 14: write37 -> write33
- U8 pad 15: latched37 -> latched33
- U8 pad 16: latched38 -> latched34
- U8 pad 17: write38 -> write34
- U8 pad 18: write39 -> write35
- U8 pad 19: latched39 -> latched35
- U8 pad 2: latched32 -> latched36
- U8 pad 3: write32 -> write36
- U8 pad 4: write33 -> write37
- U8 pad 5: latched33 -> latched37
- U8 pad 6: latched34 -> latched38
- U8 pad 7: write34 -> write38
- U8 pad 8: write35 -> write39
- U8 pad 9: latched35 -> latched39
- U9 pad 12: latched44 -> latched40
- U9 pad 13: write44 -> write40
- U9 pad 14: write45 -> write41
- U9 pad 15: latched45 -> latched41
- U9 pad 16: latched46 -> latched42
- U9 pad 17: write46 -> write42
- U9 pad 18: write47 -> write43
- U9 pad 19: latched47 -> latched43
- U9 pad 2: latched40 -> latched44
- U9 pad 3: write40 -> write44
- U9 pad 4: write41 -> write45
- U9 pad 5: latched41 -> latched45
- U9 pad 6: latched42 -> latched46
- U9 pad 7: write42 -> write46
- U9 pad 8: write43 -> write47
- U9 pad 9: latched43 -> latched47
Routing:
- net GND: track 667.4 -> 929.8 mm, vias 155 -> 202
- net write_clk: track 0.00 -> 163.2 mm, vias 0 -> 10
- net ~{ZRST}: track 0.00 -> 67.6 mm
- net +3V3: track 82.9 -> 126.8 mm, vias 14 -> 24
- net latched23: track 300.3 -> 343.7 mm, vias 3 -> 4
- net latched24: track 291.4 -> 334.2 mm, vias 3 -> 4
- net latched22: track 302.0 -> 342.3 mm, vias 3 -> 4
- net latched21: track 303.7 -> 343.0 mm, vias 3 -> 4
- net latched25: track 289.3 -> 327.8 mm, vias 3 -> 4
- net latched31: track 279.1 -> 317.5 mm, vias 3 -> 4
- net latched26: track 287.6 -> 323.9 mm, vias 3 -> 4
- net latched20: track 305.5 -> 341.6 mm, vias 3 -> 4
- net latched30: track 281.1 -> 316.8 mm, vias 3 -> 4
- net latched29: track 282.5 -> 317.4 mm, vias 3 -> 4
- net latched27: track 286.2 -> 318.4 mm, vias 3 -> 4
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