File: kdrv-discrete-pcb-register.kicad_pcb (KiCad board)
At the start: 4 copper layers, 284.3 x 65.8 mm, 215 parts, among them J1 Bus_PCI_Express_x16, J2 Bus_PCI_Express_x16, J3 Bus_PCI_Express_x16, U1 74LS00, U10 74LS273, U11 74LS273, U12 74LS541, U13 74LS541, U14 74LS541, U15 74LS541, U16 74LS541, U17 74LS541, U18 74LS541, U19 74LS541, U2 74LS00, U20 74LS04, U21 74LS30, U22 74LS541, U23 74LS541, U24 74LS541, U25 74LS541, U26 74LS541, U27 74LS541, U28 74LS541, U29 74LS541, U3 74LS30, U30 74LS04, U31 74LS30, U4 74LS273, U5 74LS273, U6 74LS273, U7 74LS273, U8 74LS273, U9 74LS273

Commit message: Finished the register board layout.  It's not as short as I would have liked, but it's done.  64 bit busses take an amount of space.
Parts:
- C3, C30, C31, U3, U31: moved to F.Cu
- moved C25 78.5 mm to (233.3, 121.2), turned to 90 degrees
- moved C29 73.9 mm to (216.5, 121.1), turned to 90 degrees
- moved C24 64.1 mm to (216.5, 121.1), turned to 90 degrees
- moved C28 57.8 mm to (199.5, 121.3), turned to 90 degrees
- moved C3 52.2 mm to (239.0, 110.7), turned to 90 degrees
- moved C23 50.9 mm to (199.5, 121.2), turned to 90 degrees
- moved C2 48.5 mm to (262.5, 110.5), turned to -90 degrees
- moved C30 48.4 mm to (160.1, 114.4), turned to -90 degrees
- moved C31 44.9 mm to (145.4, 115.3), turned to -90 degrees
- moved C26 42.9 mm to (164.9, 121.3), turned to 90 degrees
- moved C27 42.5 mm to (182.0, 121.2), turned to 90 degrees
- moved C22 41.1 mm to (182.0, 121.1), turned to 90 degrees
- moved C1 40.8 mm to (250.9, 114.2), turned to -90 degrees
- moved U2 35.6 mm to (256.8, 112.3)
- moved U3 32.6 mm to (244.9, 112.5), turned to 90 degrees
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Connections:
- U1 pad 10: /Write In/write_sel2 -> /Write In/write_sel3
- U1 pad 11: Net-(JP4-B) -> Net-(JP3-B)
- U1 pad 12: /Write In/write_sel3 -> /Write In/write_sel2
- U1 pad 13: /Write In/write_sel3 -> /Write In/write_sel2
- U1 pad 8: Net-(JP3-B) -> Net-(JP4-B)
- U1 pad 9: /Write In/write_sel2 -> /Write In/write_sel3
- U2 pad 1: /Write In/write_sel4 -> ~{write_en}
- U2 pad 11: write_clk -> Net-(JP5-B)
- U2 pad 12: Net-(U2-Pad12) -> /Write In/write_sel4
- U2 pad 13: Net-(U2-Pad12) -> /Write In/write_sel4
- U2 pad 2: /Write In/write_sel4 -> ~{write_en}
- U2 pad 3: Net-(JP5-B) -> write_en
- U2 pad 4: ~{write_en} -> Net-(U2-Pad4)
- U2 pad 5: ~{write_en} -> Net-(U2-Pad4)
- U2 pad 6: write_en -> write_clk
- U2 pad 8: Net-(U2-Pad12) -> Net-(U2-Pad4)
- U30 pad 10: Net-(JP15-B) -> Net-(JP14-B)
- U30 pad 11: /Read Out B/read_b_sel4 -> /Read Out B/read_b_sel3
- U30 pad 12: read_b_en -> Net-(JP13-B)
- U30 pad 13: ~{read_b_en} -> /Read Out B/read_b_sel2
- U30 pad 5: /Read Out B/read_b_sel2 -> ~{read_b_en}
- U30 pad 6: Net-(JP13-B) -> read_b_en
- U30 pad 8: Net-(JP14-B) -> Net-(JP15-B)
- U30 pad 9: /Read Out B/read_b_sel3 -> /Read Out B/read_b_sel4
Routing:
- net write_en: track 1.83 -> 260.3 mm
- net read_b_en: track 1.83 -> 153.5 mm
- net ~{read_b_en}: track 0.00 -> 94.7 mm, vias 0 -> 5
- net GND: track 929.8 -> 1018.9 mm, vias 202 -> 224
- net +3V3: track 126.8 -> 206.3 mm, vias 24 -> 38
- net ~{ZRST}: track 67.6 -> 138.4 mm, vias 0 -> 12
- net /Write In/write_sel0: track 0.00 -> 40.3 mm, vias 0 -> 1
- net /Write In/write_sel1: track 0.00 -> 36.4 mm
- net latched35: track 331.9 -> 298.4 mm, vias 3 -> 5
- net /Read Out B/read_b_sel0: track 0.00 -> 30.9 mm, vias 0 -> 1
- net latched34: track 333.6 -> 303.6 mm, vias 3 -> 5
- net latched33: track 335.3 -> 306.6 mm, vias 3 -> 5
- net latched36: track 330.2 -> 301.5 mm, vias 3 -> 5
- net latched32: track 337.0 -> 312.3 mm, vias 3 -> 5
- net latched37: track 328.5 -> 303.9 mm, vias 3 -> 5
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- added copper zone on In1.Cu, net +3V3
- added copper zone on In2.Cu, net GND
Other:
- board text added: "1 2 4 8 16"
- board text added: "KneeDeep RISCV Discrete Register v0.1 Daniel Williams"
- board text added: "PORTS WRITE ACTIVE READ B READ A"
- board text added: "READ B"
- board text added: "REGISTER 63 BITS 62 61 60 59 58 57 56 55 54 53 52 51 50 49 48 47 46 45 44 43 42 41 40 39 38 37 36 35 34 33 32 31 30 29 28 27 26 25 24 23 22 21 20 19 18 17 16 15 14 13 12 11 00 09 08 07 06 05 04 03 02 01 00"
- board text added: "Set register address by jumpering the address for each port. Away from the connector is a '1' bit, and toward the connector is a '0' bit."
- board text added: "The ZERO jumper is used to force the register to always produce a zero value (e.g. for the zero register). Away from the connector is 'force zero' and toward the connector is 'normal'."
- board text added: "WRITE"
- board text added: "ZERO"
